Commit message: URDF Dimensions Updated

File: navros_description/urdf/camera.xacro (robot description, xacro)
@@ -1,2 +1,26 @@
+<?xml version="1.0"?>
 <robot xmlns:xacro="http://www.ros.org/wiki/xacro" name="robot_name">
+    <joint name="camera_joint" type="fixed">
+        <parent link="base_link"/>
+        <child link="camera_link"/>
+        <origin xyz="0.0 0.0 0.0" rpy="0.0 0.0 0.0"/>
+    </joint>
+    <link name="camera_link">
+        <visual>
+            <geometry>
+                <box size="0.10 0.03 0.03"/>
+            </geometry>
+        </visual>
+    </link>
+    <joint name="camera_optical_joint" type="fixed">
+        <parent link="camera_link"/>
+        <child link="camera_link_optical"/>
+        <origin xyz="0.0 0.0 0.0" rpy="${-pi/2} 0.0 ${-pi/2}"/>
+    </joint>
+    <link name="camera_link_optical"></link>
+    <gazebo reference = "camera_link">
+        <material>
+            Gazebo/Red
+        </material>
+    </gazebo>
 </robot>

File: navros_description/urdf/navros_base.xacro (robot description, xacro)
@@ -8,9 +8,9 @@
     <!-- Wheel Radius - 35 -->
     <!-- Wheel Height - 10 -->
-    <xacro:property name="base_length" value="1.5"/>
-    <xacro:property name="base_width" value="2"/>
-    <xacro:property name="base_height" value="0.6"/>
-    <xacro:property name="wheel_radius" value="0.35"/>
-    <xacro:property name="wheel_length" value="0.1"/>
+    <xacro:property name="base_length" value="0.94"/>
+    <xacro:property name="base_width" value="1.14"/>
+    <xacro:property name="base_height" value="0.99"/>
+    <xacro:property name="wheel_radius" value="0.23"/>
+    <xacro:property name="wheel_length" value="0.05"/>
     <xacro:property name="sphere_radius" value="0.075"/>
     <link name="base_footprint"/>
@@ -85,5 +85,5 @@
         <child link="right_wheel_link"/>
         <!-- By changing the Y value, the wheel will be defined for either right or left -->
-        <origin xyz="-0.2441 -${(base_width/2) + 0.05} -0.1" rpy="0 0 0"/>
+        <origin xyz="${-(base_length/2)+ 0.15} -${(base_width/2) + 0.05} ${-(base_height/2) + 0.08}" rpy="0 0 0"/>
         <axis xyz="0 1 0"/>
     </joint>
@@ -92,5 +92,5 @@
         <child link="left_wheel_link"/>
         <!-- By changing the Y value, the wheel will be defined for either right or left -->
-        <origin xyz="-0.2441 ${(base_width/2) + 0.05} -0.1" rpy="0 0 0"/>
+        <origin xyz="${-(base_length/2)+ 0.15} ${(base_width/2) + 0.05} ${-(base_height/2) + 0.08}" rpy="0 0 0"/>
         <axis xyz="0 1 0"/>
     </joint>

Commit message: gazebo camera added

File: navros_description/urdf/camera.xacro (robot description, xacro)
@@ -4,10 +4,10 @@
         <parent link="base_link"/>
         <child link="camera_link"/>
-        <origin xyz="0.0 0.0 0.0" rpy="0.0 0.0 0.0"/>
+        <origin xyz="${base_length/2} 0 ${base_height / 2 + 0.05}" rpy="0.0 0.0 0.0"/>
     </joint>
     <link name="camera_link">
         <visual>
             <geometry>
-                <box size="0.10 0.03 0.03"/>
+                <box size="0.02 0.1 0.1"/>
             </geometry>
         </visual>
@@ -20,7 +20,25 @@
     <link name="camera_link_optical"></link>
     <gazebo reference = "camera_link">
-        <material>
-            Gazebo/Red
-        </material>
+        <material>Gazebo/Red</material>
+        <sensor name="camera" type="camera">
+            <pose> 0 0 0 0 0 0 </pose>
+            <visualize>true</visualize>
+            <update_rate>10</update_rate>
+            <camera>
+                <horizontal_fov>1.089</horizontal_fov>
+                <image>
+                    <format>R8G8B8</format>
+                    <width>640</width>
+                    <height>480</height>
+                </image>
+                <clip>
+                    <near>0.05</near>
+                    <far>8.0</far>
+                </clip>
+            </camera>
+            <plugin name="camera_controller" filename="libgazebo_ros_camera.so">
+                <frame_name>camera_link_optical</frame_name>
+            </plugin>
+        </sensor>
     </gazebo>
 </robot>
